Commit message: Fix diff-drive wheel physics so the robot actually moves.
Wheel joints now rotate around the axle, only wheels collide with the ground, and motor force is increased.

Co-authored-by: Cursor <cursoragent@cursor.com>

File: examples/diff-drive/robot/demo_mobile.urdf (robot description, URDF)
Before this commit: robot diff_drive_box, 3 links, 2 joints
Links:
- link base_link: geometry visual box size=0.7 0.3 0.5
Joints:
- joint left_wheel_joint: axis 0 1 0 -> 1 0 0
- joint right_wheel_joint: axis 0 1 0 -> 1 0 0

Commit message: Drive diff-drive robot with kinematics and follow it with the camera.
Wheel friction physics was not moving the chassis; apply diff-drive velocity from controller targets and lock pitch/roll on the base.

Co-authored-by: Cursor <cursoragent@cursor.com>

File: examples/diff-drive/robot/demo_mobile.urdf (robot description, URDF)
Before this commit: robot diff_drive_box, 3 links, 2 joints
Joints:
- joint left_wheel_joint: axis 1 0 0 -> (none); type continuous -> fixed
- joint right_wheel_joint: axis 1 0 0 -> (none); type continuous -> fixed
